Commit message: urdf changes

File: hoverboard_demo_description/urdf/hoverboard_description.xacro (robot description, xacro)
@@ -5,11 +5,11 @@
     <xacro:include filename="wheels.xacro" />
     <xacro:include filename="ros2_control.xacro" />
-    <xacro:property name="plate_radius" value="0.37" />
-    <xacro:property name="plate_height" value="0.01" />
+    <xacro:property name="plate_length" value="0.7" />
+    <xacro:property name="plate_width" value="0.4" />
+    <xacro:property name="plate_height" value="0.02" />
     <xacro:property name="chassis_weight" value="1.0" />
     <xacro:property name="driving_wheel_diameter" value="0.165" />
     <xacro:property name="driving_wheel_thickness" value="0.045" />
     <xacro:property name="driving_wheel_weight" value="2.2" />
-    <xacro:property name="driving_wheel_base_gap" value="0.01" />
     <xacro:property name="caster_wheel_diameter" value="0.09" />
     <xacro:property name="caster_wheel_weight" value="0.1" />
@@ -18,20 +18,22 @@
     <link name="plate">
         <visual>
-            <origin xyz="0 0 0" rpy="0 0 -${pi/2}"/>
+            <origin xyz="0.35 0 0.01"/>
             <geometry>
-                <mesh filename="package://hoverboard_demo_description/meshes/plate.stl" scale="0.001 0.001 0.001"/>
+                <box size="0.7 0.4 0.02"/>
             </geometry>
-            <material name="gray"/>
+            <material name="blue"/>
         </visual>
         <collision>
-            <origin xyz="0 0 0" rpy="0 0 -${pi/2}"/>
+            <origin xyz="0.35 0 0.01"/>
             <geometry>
-                <cylinder radius="${plate_radius}" length="${plate_height}"/>
+                <box size="0.7 0.4 0.02"/>
             </geometry>
         </collision>
-        <xacro:cylinder_inertia m="0.5" r="${plate_radius}" h="${plate_height}" roll="${pi/2}"/>
+        <xacro:box_inertia mass="5" x="0.7" y="0.4" z="0.02">
+            <origin xyz="0.35 0 0.01" rpy="0.0 0.0 0.0"/>
+        </xacro:box_inertia>
     </link>
     <joint name="base_link_plate_joint" type="fixed">
-        <origin rpy="0 0 0" xyz="0 0 0" />
+        <origin xyz="-0.33 0 0"/>
         <parent link="base_link" />
         <child link="plate" />
@@ -39,5 +41,4 @@
     <xacro:driving_wheel suffix="left" reflect="1"/>
     <xacro:driving_wheel suffix="right" reflect="-1"/>
-    <xacro:caster_wheel suffix="front" reflect="1" />
     <xacro:caster_wheel suffix="back" reflect="-1" />
     <xacro:hoverboard_ros2_control name="Hoverboard" />

File: hoverboard_demo_description/urdf/macros.xacro (robot description, xacro)
@@ -8,9 +8,11 @@
     </xacro:macro>
     <!-- Define some commonly used intertial properties  -->
-    <xacro:macro name="box_inertia" params="m w h d">
+    <xacro:macro name="box_inertia" params="mass x y z *origin">
         <inertial>
-            <origin xyz="0 0 0" rpy="${pi/2} 0 ${pi/2}"/>
-            <mass value="${m}"/>
-            <inertia ixx="${(m/12) * (h*h + d*d)}" ixy="0.0" ixz="0.0" iyy="${(m/12) * (w*w + d*d)}" iyz="0.0" izz="${(m/12) * (w*w + h*h)}"/>
+            <xacro:insert_block name="origin"/>
+            <mass value="${mass}" />
+            <inertia ixx="${(1/12) * mass * (y*y+z*z)}" ixy="0.0" ixz="0.0"
+                    iyy="${(1/12) * mass * (x*x+z*z)}" iyz="0.0"
+                    izz="${(1/12) * mass * (x*x+y*y)}" />
         </inertial>
     </xacro:macro>

File: hoverboard_demo_description/urdf/materials.xacro (robot description, xacro)
@@ -10,3 +10,12 @@
         <color rgba="0 0 0 1"/>
     </material>
+    <material name="green">
+        <color rgba="0 0.5 0 1" />
+    </material>
+    <material name="blue">
+        <color rgba="0.2 0.2 1 1" />
+    </material>
+    <material name="white">
+        <color rgba="1 1 1 1" />
+    </material>
 </robot>

File: hoverboard_demo_description/urdf/wheels.xacro (robot description, xacro)
@@ -24,5 +24,5 @@
             <parent link="base_link"/>
             <child link="driving_wheel_${suffix}"/>
-            <origin xyz="0 ${(plate_radius+driving_wheel_thickness+driving_wheel_base_gap-0.195)/2*reflect} 0.038" rpy="0 0 0"/>
+            <origin xyz="0 ${((plate_width/2)+driving_wheel_thickness-0.195)/2*reflect} 0.038" rpy="0 0 0"/>
         </joint>
         <gazebo reference="driving_wheel_${suffix}">

Commit message: urdf changes

File: hoverboard_demo_description/urdf/hoverboard_description.xacro (robot description, xacro)
@@ -31,9 +31,9 @@
         </collision>
         <xacro:box_inertia mass="5" x="0.7" y="0.4" z="0.02">
-            <origin xyz="0.35 0 0.01" rpy="0.0 0.0 0.0"/>
+            <origin xyz="0 0 0.01" rpy="0.0 0.0 0.0"/>
         </xacro:box_inertia>
     </link>
     <joint name="base_link_plate_joint" type="fixed">
-        <origin xyz="-0.33 0 0"/>
+        <origin xyz="0 0 0"/>
         <parent link="base_link" />
         <child link="plate" />
@@ -41,5 +41,5 @@
     <xacro:driving_wheel suffix="left" reflect="1"/>
     <xacro:driving_wheel suffix="right" reflect="-1"/>
-    <xacro:caster_wheel suffix="back" reflect="-1" />
+    <xacro:caster_wheel suffix="back" reflect="1" />
     <xacro:hoverboard_ros2_control name="Hoverboard" />
 </robot>

File: hoverboard_demo_description/urdf/wheels.xacro (robot description, xacro)
@@ -24,5 +24,5 @@
             <parent link="base_link"/>
             <child link="driving_wheel_${suffix}"/>
-            <origin xyz="0 ${((plate_width/2)+driving_wheel_thickness-0.195)/2*reflect} 0.038" rpy="0 0 0"/>
+            <origin xyz="0 ${0.26*reflect} 0.0" rpy="0 0 0"/>
         </joint>
         <gazebo reference="driving_wheel_${suffix}">
@@ -56,5 +56,5 @@
             <parent link="base_link"/>
             <child link="caster_wheel_${suffix}"/>
-            <origin xyz="${0.12*reflect} 0 0" rpy="0 0 0"/>
+            <origin xyz="0.7 0 0" rpy="0 0 0"/>
         </joint>
         <gazebo reference="caster_wheel_${suffix}">
