Commit message: bring hoverboard up to current.

File: urdf/gps.xacro (robot description, xacro)
@@ -2,7 +2,7 @@
 <robot name="hoverboard_robot" xmlns:xacro="http://ros.org/wiki/xacro">
     <joint name="gps_joint" type="fixed">
-        <parent link="plate"/>
+        <parent link="base_link"/>
         <child link="gps"/>
-        <origin xyz="-0.2 0 0.1" rpy="0 0 0"/>
+        <origin xyz="0.2 0 0.1" rpy="0 0 0"/>
     </joint>
     <link name="gps">

File: urdf/hoverboard_description.xacro (robot description, xacro)
@@ -7,5 +7,5 @@
     <xacro:include filename="lidar.xacro" />
     <xacro:include filename="gps.xacro" />
-    <xacro:include filename="mag.xacro" />
+    <xacro:include filename="imu.xacro" />
     <xacro:property name="plate_length" value="0.7" />
     <xacro:property name="plate_width" value="0.4" />
@@ -23,5 +23,5 @@
             <origin xyz="0.35 0 0.01"/>
             <geometry>
-                <box size="0.7 0.4 0.02"/>
+                <box size="0.7 0.5 0.02"/>
             </geometry>
             <material name="blue"/>
@@ -38,7 +38,14 @@
     </link>
     <joint name="base_link_plate_joint" type="fixed">
+        <origin xyz="-0.08255 0 0"/>
+        <parent link="base_link" />
+        <child link="plate" />
+    </joint>
+    <link name="base_footprint">
+    </link>
+    <joint name="base_footprint_joint" type="fixed">
         <origin xyz="0 0 0"/>
         <parent link="base_link" />
-        <child link="plate" />
+        <child link="base_footprint" />
     </joint>
     <xacro:driving_wheel suffix="left" reflect="1"/>

File: urdf/imu.xacro (robot description, xacro)
@@ -1,15 +1,15 @@
 <?xml version="1.0"?>
 <robot name="hoverboard_robot" xmlns:xacro="http://ros.org/wiki/xacro">
-    <joint name="magnetometer_link_joint" type="fixed">
-        <parent link="plate"/>
-        <child link="magnetometer_link"/>
-        <origin xyz="0 0 0" rpy="0 0 0"/>
+    <joint name="imu_link_joint" type="fixed">
+        <parent link="base_link"/>
+        <child link="imu_link"/>
+        <origin xyz="0.05 0 0.02" rpy="0 0 ${pi}"/>
     </joint>
-    <link name="magnetometer_link">
+    <link name="imu_link">
         <visual>
             <geometry>
                 <box size="0.02 0.02 0.01"/>
             </geometry>
-            <material name="blue"/>
+            <material name="red"/>
         </visual>
         <collision>

File: urdf/lidar.xacro (robot description, xacro)
@@ -2,7 +2,7 @@
 <robot name="hoverboard_robot" xmlns:xacro="http://ros.org/wiki/xacro">
     <joint name="laser_joint" type="fixed">
-        <parent link="plate"/>
+        <parent link="base_link"/>
         <child link="laser"/>
-        <origin xyz="0 0 0.1" rpy="0 0 0"/>
+        <origin xyz="0 0 0.1" rpy="0 0 ${pi}"/>
     </joint>
     <link name="laser">

File: urdf/materials.xacro (robot description, xacro)
@@ -13,4 +13,7 @@
         <color rgba="0 0.5 0 1" />
     </material>
+    <material name="red">
+        <color rgba="0.5 0 0 1" />
+    </material>
     <material name="blue">
         <color rgba="0.2 0.2 1 1" />

File: urdf/ros2_control.xacro (robot description, xacro)
@@ -8,5 +8,5 @@
         <param name="right_wheel_joint_name">driving_wheel_right_joint</param>
         <param name="loop_rate">50</param>
-        <param name="device">/dev/ttyS0</param>
+        <param name="device">/dev/ttyTHS1</param>
         <param name="baud_rate">115200</param>
         <param name="timeout">1000</param>

File: urdf/wheels.xacro (robot description, xacro)
@@ -56,5 +56,5 @@
             <parent link="base_link"/>
             <child link="caster_wheel_${suffix}"/>
-            <origin xyz="0.7 0 0" rpy="0 0 0"/>
+            <origin xyz="0.6 0 0" rpy="0 0 0"/>
         </joint>
         <gazebo reference="caster_wheel_${suffix}">
